File: pcb/FTDI-Breakout_v20.brd (EAGLE design)
At the start: 30 x 16 mm, 35 parts, among them IC1 FT231XQ, IC2 LDO-TS5204-3V3, X1 PASSER-07, X2 PASSER-07

Commit message: updated schematics and layout
Connections:
- net GND: now also IC1.TP; no longer IC1.PAD
Changed lines of the file:
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@@
 <layer number="154" name="FabDoc2" color="2" fill="1" visible="no" active="no"/>
 <layer number="155" name="FabDoc3" color="7" fill="15" visible="no" active="no"/>
+<layer number="200" name="200bmp" color="1" fill="10" visible="no" active="no"/>
 <layer number="217" name="217bmp" color="18" fill="1" visible="no" active="no"/>
 <layer number="218" name="218bmp" color="19" fill="1" visible="no" active="no"/>
@@
 <attribute name="NAME" x="11.27125" y="15.24" size="0.8128" layer="25" font="vector" ratio="10" rot="R180" align="center"/>
 <attribute name="VALUE" x="11.27125" y="12.85875" size="0.8128" layer="27" font="vector" ratio="10" rot="R180" align="center"/>
+<attribute name="NRND" value="NRND" x="11.27125" y="12.85875" size="1.778" layer="27" rot="R270" display="off"/>
 </element>
 <element name="F1" library="we-rcl" package="R0805" value="0.5A" x="7.62" y="10.31875" smashed="yes" rot="R90">
@@
 <signal name="GND">
 <contactref element="IC1" pad="13"/>
-<contactref element="IC1" pad="PAD"/>
+<contactref element="IC1" pad="TP"/>
 <contactref element="IC1" pad="3"/>
 <contactref element="IC2" pad="3"/>

Commit message: updated layout and schematics
Parts:
- C1, C3, C4, C6, C7, C8, C9, CU, R1, R2, R3, R4, R5, R6, R7, R8, RU: device we-rcl:R0603 -> we-rcl:C0603
- C2, C5, F1: device we-rcl:R0805 -> we-rcl:C0805
- RX, TX: value LED-0603 -> (none); device we-opto:LED_0603 -> we-opto:C0603
