File: pcb/FTDI-Breakout_v20.sch (EAGLE design)
At the start: 35 parts, among them IC1 FT231XQ, IC2 LDO-TS5204-3V3, X1 PASSER-07, X2 PASSER-07

Commit message: updated schematics and layout
Changed lines of the file:
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@@
 <layer number="154" name="FabDoc2" color="2" fill="1" visible="no" active="no"/>
 <layer number="155" name="FabDoc3" color="7" fill="15" visible="no" active="no"/>
+<layer number="200" name="200bmp" color="1" fill="10" visible="no" active="no"/>
 <layer number="217" name="217bmp" color="18" fill="1" visible="no" active="no"/>
 <layer number="218" name="218bmp" color="19" fill="1" visible="no" active="no"/>

Commit message: cleaned up schematics and layout
Other:
- note removed: "www.watterott.com"
Changed lines of the file:
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@@
 <setting verticaltext="up"/>
 </settings>
-<grid distance="0.1" unitdist="inch" unit="inch" style="lines" multiple="1" display="no" altdistance="0.01" altunitdist="inch" altunit="inch"/>
+<grid distance="0.05" unitdist="inch" unit="inch" style="lines" multiple="1" display="yes" altdistance="0.025" altunitdist="inch" altunit="inch"/>
 <layers>
 <layer number="1" name="Top" color="4" fill="1" visible="no" active="no"/>
@@
 <sheet>
 <plain>
-<text x="213.36" y="5.08" size="2.54" layer="94" font="vector" align="bottom-right">www.watterott.com</text>
-<text x="161.29" y="31.75" size="1.27" layer="95">Released under the Creative Commons Attribution Share-Alike License</text>
-<text x="161.29" y="29.21" size="1.27" layer="95">http://creativecommons.org/licenses/by-sa/4.0/</text>
-<text x="161.29" y="25.4" size="1.27" layer="95">Designed by Andreas Watterott (Watterott electronic)</text>
+<text x="162.56" y="21.59" size="1.27" layer="95">Released under the Creative Commons Attribution Share-Alike License</text>
+<text x="162.56" y="19.05" size="1.27" layer="95">http://creativecommons.org/licenses/by-sa/4.0/</text>
+<text x="162.56" y="15.24" size="1.27" layer="95">Designed by Andreas Watterott (Watterott electronic)</text>
 <text x="76.2" y="111.76" size="1.778" layer="94" align="top-right">Option 1: RU= 0, CU=NC
 Option 2: RU=330, CU=100n</text>
@@
 <instances>
 <instance part="FRAME1" gate="G$1" x="0" y="0"/>
-<instance part="LOGO2" gate="G$1" x="207.01" y="19.05"/>
-<instance part="X1" gate="X" x="166.37" y="19.05"/>
-<instance part="X2" gate="X" x="173.99" y="19.05"/>
+<instance part="LOGO2" gate="G$1" x="187.96" y="7.62"/>
+<instance part="X1" gate="X" x="165.1" y="7.62"/>
+<instance part="X2" gate="X" x="170.18" y="7.62"/>
 <instance part="IC1" gate="IC" x="166.37" y="128.27"/>
 <instance part="IC2" gate="A" x="81.28" y="62.23"/>
@@
 <instance part="C7" gate="C" x="111.76" y="130.81" rot="R90"/>
 <instance part="GND1" gate="1" x="106.68" y="125.73"/>
-<instance part="LOGO1" gate="G$1" x="193.04" y="19.05"/>
-<instance part="LOGO4" gate="G$1" x="207.01" y="11.43"/>
-<instance part="LOGO3" gate="G$1" x="193.04" y="11.43"/>
+<instance part="LOGO1" gate="G$1" x="177.8" y="7.62"/>
+<instance part="LOGO4" gate="G$1" x="208.28" y="7.62"/>
+<instance part="LOGO3" gate="G$1" x="198.12" y="7.62"/>
 </instances>
 <busses>

Commit message: updated layout and schematics
Parts:
- C1, C3, C4, C6, C7, C8, C9, CU: device we-rcl:CAPACITOR-C0603 -> we-rcl:CAPACITOR-0603
- C2, C5: device we-rcl:CAPACITOR-C0805 -> we-rcl:CAPACITOR-0805
- R1, R2, R3, R4, R5, R6, R7, R8, RU: device we-rcl:RESISTOR-R0603 -> we-rcl:RESISTOR-0603
- RX, TX: value LED-0603 -> (none)
Connections:
- net CBUS1: now also IC1.RXLED/CBUS1; no longer IC1.CBUS1
- net CBUS2: now also IC1.TXLED/CBUS2; no longer IC1.CBUS2
Changed lines of the file:
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@@
 <?xml version="1.0" encoding="utf-8"?>
 <!DOCTYPE eagle SYSTEM "eagle.dtd">
-<eagle version="6.6.0">
+<eagle version="7.2.0">
 <drawing>
 <settings>
@@
 <part name="FTDI" library="we-board" deviceset="FTDI" device=""/>
 <part name="SW" library="we-switch" deviceset="SW-2UM" device="-CUS22B"/>
-<part name="R5" library="we-rcl" deviceset="RESISTOR" device="-R0603" value="27"/>
-<part name="R6" library="we-rcl" deviceset="RESISTOR" device="-R0603" value="27"/>
-<part name="R7" library="we-rcl" deviceset="RESISTOR" device="-R0603" value="27"/>
-<part name="R8" library="we-rcl" deviceset="RESISTOR" device="-R0603" value="27"/>
+<part name="R5" library="we-rcl" deviceset="RESISTOR" device="-0603" value="27"/>
+<part name="R6" library="we-rcl" deviceset="RESISTOR" device="-0603" value="27"/>
+<part name="R7" library="we-rcl" deviceset="RESISTOR" device="-0603" value="27"/>
+<part name="R8" library="we-rcl" deviceset="RESISTOR" device="-0603" value="27"/>
 <part name="GND10" library="supply1" deviceset="GND" device=""/>
 <part name="+3V2" library="supply1" deviceset="+3V3" device=""/>
 <part name="P+11" library="supply1" deviceset="+5V" device=""/>
-<part name="C3" library="we-rcl" deviceset="CAPACITOR" device="-C0603" value="100n"/>
-<part name="C4" library="we-rcl" deviceset="CAPACITOR" device="-C0603" value="100n"/>
-<part name="C5" library="we-rcl" deviceset="CAPACITOR" device="-C0805" value="4u7"/>
-<part name="R1" library="we-rcl" deviceset="RESISTOR" device="-R0603" value="27"/>
-<part name="R2" library="we-rcl" deviceset="RESISTOR" device="-R0603" value="27"/>
-<part name="C1" library="we-rcl" deviceset="CAPACITOR" device="-C0603" value="10n"/>
-<part name="CU" library="we-rcl" deviceset="CAPACITOR" device="-C0603" value="NC"/>
-<part name="RU" library="we-rcl" deviceset="RESISTOR" device="-R0603" value="0"/>
+<part name="C3" library="we-rcl" deviceset="CAPACITOR" device="-0603" value="100n"/>
+<part name="C4" library="we-rcl" deviceset="CAPACITOR" device="-0603" value="100n"/>
+<part name="C5" library="we-rcl" deviceset="CAPACITOR" device="-0805" value="4u7"/>
+<part name="R1" library="we-rcl" deviceset="RESISTOR" device="-0603" value="27"/>
+<part name="R2" library="we-rcl" deviceset="RESISTOR" device="-0603" value="27"/>
+<part name="C1" library="we-rcl" deviceset="CAPACITOR" device="-0603" value="10n"/>
+<part name="CU" library="we-rcl" deviceset="CAPACITOR" device="-0603" value="NC"/>
+<part name="RU" library="we-rcl" deviceset="RESISTOR" device="-0603" value="0"/>
 <part name="RX" library="we-opto" deviceset="LED" device="-0603"/>
-<part name="R3" library="we-rcl" deviceset="RESISTOR" device="-R0603" value="1k"/>
+<part name="R3" library="we-rcl" deviceset="RESISTOR" device="-0603" value="1k"/>
 <part name="TX" library="we-opto" deviceset="LED" device="-0603"/>
-<part name="R4" library="we-rcl" deviceset="RESISTOR" device="-R0603" value="1k"/>
-<part name="C8" library="we-rcl" deviceset="CAPACITOR" device="-C0603" value="100n"/>
-<part name="C9" library="we-rcl" deviceset="CAPACITOR" device="-C0603" value="100n"/>
-<part name="C2" library="we-rcl" deviceset="CAPACITOR" device="-C0805" value="4u7"/>
+<part name="R4" library="we-rcl" deviceset="RESISTOR" device="-0603" value="1k"/>
+<part name="C8" library="we-rcl" deviceset="CAPACITOR" device="-0603" value="100n"/>
+<part name="C9" library="we-rcl" deviceset="CAPACITOR" device="-0603" value="100n"/>
+<part name="C2" library="we-rcl" deviceset="CAPACITOR" device="-0805" value="4u7"/>
 <part name="CBUS0" library="we-rcl" deviceset="PAD" device="-1.27X1.27_NC" value="PAD-1.27X1.27_NC"/>
 <part name="CBUS3" library="we-rcl" deviceset="PAD" device="-1.27X1.27_NC" value="PAD-1.27X1.27_NC"/>
-<part name="C6" library="we-rcl" deviceset="CAPACITOR" device="-C0603" value="47p"/>
-<part name="C7" library="we-rcl" deviceset="CAPACITOR" device="-C0603" value="47p"/>
+<part name="C6" library="we-rcl" deviceset="CAPACITOR" device="-0603" value="47p"/>
+<part name="C7" library="we-rcl" deviceset="CAPACITOR" device="-0603" value="47p"/>
 <part name="GND1" library="supply1" deviceset="GND" device=""/>
 <part name="LOGO1" library="we-symbol" deviceset="WEEE_LOGO" device="-S"/>
@@
 </plain>
 <instances>
-<instance part="FRAME1" gate="G$1" x="0" y="0"/>
-<instance part="LOGO2" gate="G$1" x="187.96" y="7.62"/>
+<instance part="FRAME1" gate="F" x="0" y="0"/>
+<instance part="LOGO2" gate="L" x="187.96" y="7.62"/>
 <instance part="X1" gate="X" x="165.1" y="7.62"/>
 <instance part="X2" gate="X" x="170.18" y="7.62"/>
@@
 <attribute name="VALUE" x="68.58" y="123.19" size="1.778" layer="96" align="top-center"/>
 </instance>
-<instance part="RX" gate="L" x="171.45" y="96.52" rot="R90"/>
+<instance part="RX" gate="D" x="171.45" y="96.52" rot="R90"/>
 <instance part="R3" gate="R" x="161.29" y="96.52" rot="R180"/>
-<instance part="TX" gate="L" x="171.45" y="86.36" rot="R90"/>
+<instance part="TX" gate="D" x="171.45" y="86.36" rot="R90"/>
 <instance part="R4" gate="R" x="161.29" y="86.36" rot="R180"/>
 <instance part="C8" gate="C" x="132.08" y="114.3" rot="R90"/>
@@
 <instance part="C7" gate="C" x="111.76" y="130.81" rot="R90"/>
 <instance part="GND1" gate="1" x="106.68" y="125.73"/>
-<instance part="LOGO1" gate="G$1" x="177.8" y="7.62"/>
-<instance part="LOGO4" gate="G$1" x="208.28" y="7.62"/>
-<instance part="LOGO3" gate="G$1" x="198.12" y="7.62"/>
+<instance part="LOGO1" gate="L" x="177.8" y="7.62"/>
+<instance part="LOGO4" gate="L" x="208.28" y="7.62"/>
+<instance part="LOGO3" gate="L" x="198.12" y="7.62"/>
 </instances>
 <busses>
@@
 <net name="CBUS1" class="0">
 <segment>
-<pinref part="IC1" gate="IC" pin="CBUS1"/>
+<pinref part="IC1" gate="IC" pin="RXLED/CBUS1"/>
 <label x="189.23" y="118.11" size="1.27" layer="95" xref="yes"/>
 <wire x1="189.23" y1="118.11" x2="184.15" y2="118.11" width="0.1524" layer="91"/>
 </segment>
 <segment>
-<pinref part="RX" gate="L" pin="C"/>
+<pinref part="RX" gate="D" pin="C"/>
 <wire x1="181.61" y1="96.52" x2="176.53" y2="96.52" width="0.1524" layer="91"/>
 <label x="181.61" y="96.52" size="1.27" layer="95" xref="yes"/>
@@
 <net name="CBUS2" class="0">
 <segment>
-<pinref part="IC1" gate="IC" pin="CBUS2"/>
+<pinref part="IC1" gate="IC" pin="TXLED/CBUS2"/>
 <label x="189.23" y="115.57" size="1.27" layer="95" xref="yes"/>
 <wire x1="184.15" y1="115.57" x2="189.23" y2="115.57" width="0.1524" layer="91"/>
 </segment>
 <segment>
-<pinref part="TX" gate="L" pin="C"/>
+<pinref part="TX" gate="D" pin="C"/>
 <wire x1="181.61" y1="86.36" x2="176.53" y2="86.36" width="0.1524" layer="91"/>
 <label x="181.61" y="86.36" size="1.27" layer="95" xref="yes"/>
@@
 <net name="RX-LED" class="0">
 <segment>
-<pinref part="RX" gate="L" pin="A"/>
+<pinref part="RX" gate="D" pin="A"/>
 <pinref part="R3" gate="R" pin="1"/>
 <wire x1="166.37" y1="96.52" x2="168.91" y2="96.52" width="0.1524" layer="91"/>
@@
 <net name="TX-LED" class="0">
 <segment>
-<pinref part="TX" gate="L" pin="A"/>
+<pinref part="TX" gate="D" pin="A"/>
 <pinref part="R4" gate="R" pin="1"/>
 <wire x1="166.37" y1="86.36" x2="168.91" y2="86.36" width="0.1524" layer="91"/>
